Commit message: mapas

File: my_bot/description/robot_core.xacro (robot description, xacro)
@@ -5,10 +5,10 @@
     <xacro:property name="chassis_width" value="0.19"/>
     <xacro:property name="chassis_height" value="0.02"/>
-    <xacro:property name="chassis_mass" value="2"/>
+    <xacro:property name="chassis_mass" value="2.0"/>
     <xacro:property name="wheel_radius" value="0.03325"/>
     <xacro:property name="wheel_thickness" value="0.0266"/>
     <xacro:property name="wheel_mass" value="0.03"/>
     <xacro:property name="wheel_offset_x" value="0.02"/>
-    <xacro:property name="wheel_offset_y" value="0.11"/>
+    <xacro:property name="wheel_offset_y" value="0.13"/>
     <xacro:property name="wheel_offset_z" value="0"/>
     <xacro:property name="caster_wheel_radius" value="0.02"/>
