Commit message: ultimos ajustes

File: my_bot/description/lidar.xacro (robot description, xacro)
@@ -4,5 +4,5 @@
         <parent link="chassis"/>
         <child link="laser_frame"/>
-        <origin xyz="0.122 0 0.212" rpy="0 0 0"/>
+         <origin xyz="0.08 0 0.212" rpy="0 0 0"/> <!--0.122-->
     </joint>
     <link name="laser_frame">

File: my_bot/description/robot_core.xacro (robot description, xacro)
@@ -2,7 +2,7 @@
 <robot xmlns:xacro="http://www.ros.org/wiki/xacro" >
     <xacro:include filename="inertial_macros.xacro"/>
-    <xacro:property name="chassis_length" value="0.23"/>
+    <xacro:property name="chassis_length" value="0.28"/> <!--0.23-->
     <xacro:property name="chassis_width" value="0.19"/>
-    <xacro:property name="chassis_height" value="0.02"/>
+    <xacro:property name="chassis_height" value="0.15"/>
     <xacro:property name="chassis_mass" value="2.0"/>
     <xacro:property name="wheel_radius" value="0.03325"/>
@@ -10,5 +10,5 @@
     <xacro:property name="wheel_mass" value="0.03"/>
     <xacro:property name="wheel_offset_x" value="0.02"/>
-    <xacro:property name="wheel_offset_y" value="0.13"/>
+    <xacro:property name="wheel_offset_y" value="0.125"/>
     <xacro:property name="wheel_offset_z" value="0"/>
     <xacro:property name="caster_wheel_radius" value="0.02"/>

File: my_bot/description/ros2_control.xacro (robot description, xacro)
@@ -6,9 +6,9 @@
                 <param name="left_wheel_name">left_wheel_joint</param>
                 <param name="right_wheel_name">right_wheel_joint</param>
-                <param name="loop_rate">30</param>
+                <param name="loop_rate">100</param>
                 <param name="device">/dev/ttyACM0</param>
                 <param name="baud_rate">115200</param>
-                <param name="timeout">5000</param>
-                <param name="enc_counts_per_rev">1300</param>
+                <param name="timeout">10000</param>
+                <param name="enc_counts_per_rev">620</param>
             </hardware>
             <joint name="left_wheel_joint">
